Commit message: fix(dm): widen gripper finger travel to 50mm (100mm total opening)
Sync DM URDF finger limits with the simulator repo: finger_left upper
0.0285 -> 0.05, finger_right lower -0.0285 -> -0.05.

File: DM/urdf/ReBot_Arm_DM.urdf (robot description, URDF)
Before this commit: robot ReBot_Arm_DM, 10 links, 9 joints
Joints:
- joint finger_left: limit lower=0 upper=0.0285 effort=8 velocity=0.08 -> lower=0 upper=0.05 effort=8 velocity=0.08
- joint finger_right: limit lower=-0.0285 upper=0 effort=8 velocity=0.08 -> lower=-0.05 upper=0 effort=8 velocity=0.08
